Commit message: dy_ob

File: src/robot_simulator/urdf/car.urdf.xacro (robot description, xacro)
@@ -1,4 +1,5 @@
 <robot name="mycar" xmlns:xacro="http://www.ros.org/wiki/xacro">
  <xacro:property name="cmd_vel_top" value="$(arg cmd_vel_top)"/>
+ <xacro:property name="odom_top" value="$(arg odom_top)"/>
     <xacro:include filename="head.xacro" />
     <xacro:include filename="demo05_car_base.urdf.xacro" />
@@ -7,4 +8,5 @@
     <xacro:include filename="gazebo/move.xacro"  >
         <xacro:property name="cmd_vel_top" value="$(cmd_vel_top)"/>
+         <xacro:property name="odom_top" value="$(odom_top)"/>
     </xacro:include>
     <!-- <xacro:include filename="gazebo/laser.xacro" /> -->

File: src/robot_simulator/urdf/gazebo/move.xacro (robot description, xacro)
@@ -16,5 +16,4 @@
     <xacro:joint_trans joint_name="left_wheel2base_link" />
     <xacro:joint_trans joint_name="right_wheel2base_link" />
-<!-- <xacro:property name="cmd_vel_top" value="$(cmd_vel_top1)"/> -->
     <gazebo>
         <plugin name="differential_drive_controller" filename="libgazebo_ros_diff_drive.so">
@@ -36,5 +35,5 @@
             <!-- <publishOdomTF>true</publishOdomTF>   -->
             <odometryFrame>map</odometryFrame>
-            <odometryTopic>odom1</odometryTopic>
+            <odometryTopic>${odom_top}</odometryTopic>
             <robotBaseFrame>base_footprint_obs</robotBaseFrame>
         </plugin>

Commit message: add prediction and cp in ssc_map.py

File: src/robot_simulator/urdf/car.urdf.xacro (robot description, xacro)
@@ -2,11 +2,15 @@
  <xacro:property name="cmd_vel_top" value="$(arg cmd_vel_top)"/>
  <xacro:property name="odom_top" value="$(arg odom_top)"/>
+<xacro:property name="base_name" value="$(arg base_name)"/>
     <xacro:include filename="head.xacro" />
-    <xacro:include filename="demo05_car_base.urdf.xacro" />
-    <!-- <xacro:include filename="demo06_car_camera.urdf.xacro" /> -->
+    <xacro:include filename="demo05_car_base.urdf.xacro" >
+         <xacro:property name="base_name" value="$(base_name)"/>
+     </xacro:include>
+    <!-- <xacro:include filename="demo06_car_camera.urdf.xazcro" /> -->
     <!-- <xacro:include filename="demo07_car_laser.urdf.xacro" /> -->
     <xacro:include filename="gazebo/move.xacro"  >
         <xacro:property name="cmd_vel_top" value="$(cmd_vel_top)"/>
          <xacro:property name="odom_top" value="$(odom_top)"/>
+         <xacro:property name="base_name" value="$(base_name)"/>
     </xacro:include>
     <!-- <xacro:include filename="gazebo/laser.xacro" /> -->

File: src/robot_simulator/urdf/demo05_car_base.urdf.xacro (robot description, xacro)
@@ -8,4 +8,5 @@
     <xacro:property name="base_link_length" value="0.08" />
     <xacro:property name="base_link_m" value="0.5" />
+    <xacro:property name="base_name" value="$(arg base_name)"/>  <!--base_footprint_obs-->
 <xacro:property name="earth_space" value="0.015" />
     <xacro:include filename="$(find velodyne_description)/urdf/VLP-16.urdf.xacro"/>
@@ -17,5 +18,5 @@
         <origin xyz="0 0 0.5" rpy="0 0 0" />
     </HDL-32E> -->
-    <link name="base_footprint_obs">
+    <link name="${base_name}">
       <visual>
         <geometry>
@@ -46,5 +47,5 @@
     </gazebo>
     <joint name="base_link2base_footprint_obs" type="fixed">
-      <parent link="base_footprint_obs" />
+      <parent link="${base_name}" />
       <child link="base_link" />
       <origin xyz="0 0 ${earth_space + base_link_length / 2 }" rpy="0 0 0" />
@@ -64,5 +65,5 @@
         <xyzOffset>0 0 0</xyzOffset>
         <rpyOffset>0 0 0</rpyOffset>
-        <frameName>base_footprint_obs</frameName>
+        <frameName>${base_name}</frameName>
         <initialOrientationAsReference>false</initialOrientationAsReference>
       </plugin>

File: src/robot_simulator/urdf/gazebo/move.xacro (robot description, xacro)
@@ -36,5 +36,5 @@
             <odometryFrame>map</odometryFrame>
             <odometryTopic>${odom_top}</odometryTopic>
-            <robotBaseFrame>base_footprint_obs</robotBaseFrame>
+            <robotBaseFrame>${base_name}</robotBaseFrame>
         </plugin>
     </gazebo>
